File: td-io.kicad_sch (KiCad schematic)
At the start: 18 parts, among them J1 USB_B, J2 I2C, J3 Dips, J4 Test/Service, J5 Power, J6 Control IO, Q1 AO4818B, Q2 AO3400A, U1 ISL3175EIBZ-T, U2 Pico

Commit message: Minor fixes
Parts:
- J6: value Control IO -> Controls
Changed lines of the file:
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@@
       (effects (font (size 1.27 1.27)) (justify right))
     )
-    (property "Value" "Control IO" (id 1) (at 349.25 246.38 90)
+    (property "Value" "Controls" (id 1) (at 349.25 246.38 90)
       (effects (font (size 1.27 1.27)) (justify right))
     )
@@
     )
     (path "/51cf508d-59ed-43ac-92da-b1be242395a6"
-      (reference "J6") (unit 1) (value "Control IO") (footprint "Connector_PinHeader_2.54mm:PinHeader_2x10_P2.54mm_Vertical")
+      (reference "J6") (unit 1) (value "Controls") (footprint "Connector_PinHeader_2.54mm:PinHeader_2x10_P2.54mm_Vertical")
     )
     (path "/00000000-0000-0000-0000-000060ff630d"
