File: td-io.kicad_sch (KiCad schematic)
At the start: 18 parts, among them J1 USB_B, J2 I2C, J3 Dips, J4 Test/Service, J5 Power, J6 Controls, Q1 AO4818B, Q2 AO3400A, U1 ISL3175EIBZ-T, U2 Pico

Commit message: misc stuff
Parts:
- removed D1: BAV99S, Package_TO_SOT_SMD:SOT-363_SC-70-6, symbol Diode:BAV99S
- removed J2: I2C, Connector_PinHeader_2.54mm:PinHeader_1x02_P2.54mm_Vertical, symbol Connector_Generic:Conn_01x02
- removed J3: Dips, Connector_PinHeader_2.54mm:PinHeader_1x03_P2.54mm_Vertical, symbol Connector_Generic:Conn_01x03
- removed J4: Test/Service, Connector_PinHeader_2.54mm:PinHeader_1x03_P2.54mm_Vertical, symbol Connector_Generic:Conn_01x03
- removed Q1: AO4818B, Package_SO:SOIC-8_3.9x4.9mm_P1.27mm, symbol Transistor_FET:FDS6930B
- added J2: Misc, Connector_JST:JST_PH_B4B-PH-K_1x04_P2.00mm_Vertical, symbol Connector_Generic:Conn_01x04
- added J3: Dips, Connector_JST:JST_PH_B4B-PH-K_1x04_P2.00mm_Vertical, symbol Connector_Generic:Conn_01x04
- H1, H2, H3, H4: footprint MountingHole:MountingHole_3.5mm_Pad -> MountingHole:MountingHole_2.5mm_Pad
- J5: footprint Connector_PinHeader_2.54mm:PinHeader_1x02_P2.54mm_Vertical -> Connector_JST:JST_XH_B2B-XH-AM_1x02_P2.50mm_Vertical
- R2: value 100 -> 1k
- R3: value 10k -> 1k
- renumbered Q2 to Q1
Connections:
- net GND: now also R2.2, J2.4 (Pin_4), J3.4 (Pin_4); no longer H1.1, H2.1, H3.1, H4.1
- net b_coin: now also J2.1 (Pin_1)
- net b_service: now also J2.3 (Pin_3)
- net b_test: now also J2.2 (Pin_2)
- net dip1: now also U2.7 (GPIO5), J3.1 (Pin_1); no longer J6.11 (Pin_11), U2.15 (GPIO11)
- net dip2: now also J6.11 (Pin_11), U2.15 (GPIO11), J3.2 (Pin_2); no longer J6.16 (Pin_16), U2.16 (GPIO12)
- net dip3: now also J6.16 (Pin_16), U2.16 (GPIO12), J3.3 (Pin_3)
- no-connect marks 13 -> 14
Other:
- note removed: "AO4818B is only here for legacy reasons and should not be placed if AO3400A is placed."
- moved on the sheet: H1, H2, H3, H4, J5
